File: control_logic.kicad_sch (KiCad schematic)
At the start: 5 parts, among them J1 Conn_01x24, J2 Conn_01x24, U1 ESP32-S3-WROOM-1

Commit message: Added some fan safety
Parts:
- added R54: 100k, symbol Device:R
Connections:
- net +3.3V: now also R54.1
- net MUTE_3V3: now also R54.2
- net TACHOMETER: now reaches U1.24 (IO47)
Other:
- sheet PCB_Fan ports: added TACHOMETER; removed none
Changed lines of the file:
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@@
 		(color 0 0 0 0)
 	)
+	(junction
+		(at 29.21 152.4)
+		(diameter 0)
+		(color 0 0 0 0)
+	)
 	(wire
 		(pts
@@
 	(wire
 		(pts
+			(xy 198.12 149.86) (xy 203.2 149.86)
+		)
+		(stroke
+			(width 0)
+			(type default)
+		)
+	)
+	(wire
+		(pts
+			(xy 27.94 152.4) (xy 29.21 152.4)
+		)
+		(stroke
+			(width 0)
+			(type default)
+		)
+	)
+	(wire
+		(pts
+			(xy 17.78 152.4) (xy 20.32 152.4)
+		)
+		(stroke
+			(width 0)
+			(type default)
+		)
+	)
+	(wire
+		(pts
 			(xy 43.18 140.97) (xy 43.18 144.78)
 		)
@@
 	(wire
 		(pts
+			(xy 29.21 152.4) (xy 44.45 152.4)
+		)
+		(stroke
+			(width 0)
+			(type default)
+		)
+	)
+	(wire
+		(pts
 			(xy 162.56 99.06) (xy 167.64 99.06)
 		)
@@
 	(wire
 		(pts
+			(xy 26.67 157.48) (xy 29.21 157.48)
+		)
+		(stroke
+			(width 0)
+			(type default)
+		)
+	)
+	(wire
+		(pts
 			(xy 162.56 40.64) (xy 167.64 40.64)
+		)
+		(stroke
+			(width 0)
+			(type default)
+		)
+	)
+	(wire
+		(pts
+			(xy 29.21 157.48) (xy 29.21 152.4)
 		)
 		(stroke
@@
 		)
 	)
+	(label "TACHOMETER"
+		(at 74.93 187.96 0)
+		(effects
+			(font
+				(size 1.27 1.27)
+			)
+			(justify left)
+		)
+	)
 	(label "FPGA_TO_MCU"
 		(at 74.93 147.32 0)
@@
 		)
 	)
+	(label "TACHOMETER"
+		(at 198.12 149.86 180)
+		(effects
+			(font
+				(size 1.27 1.27)
+			)
+			(justify right)
+		)
+	)
 	(label "DAC_DATA_34"
 		(at 111.76 88.9 0)
@@
 	)
 	(label "MUTE_3V3"
-		(at 44.45 152.4 180)
+		(at 26.67 157.48 180)
 		(effects
 			(font
@@
 	)
 	(symbol
+		(lib_id "Device:R")
+		(at 24.13 152.4 90)
+		(unit 1)
+		(exclude_from_sim no)
+		(in_bom yes)
+		(on_board yes)
+		(dnp no)
+		(fields_autoplaced yes)
+		(property "Reference" "R54"
+			(at 24.13 146.05 90)
+			(effects
+				(font
+					(size 1.27 1.27)
+				)
+			)
+		)
+		(property "Value" "100k"
+			(at 24.13 148.59 90)
+			(effects
+				(font
+					(size 1.27 1.27)
+				)
+			)
+		)
+		(property "Footprint" ""
+			(at 24.13 154.178 90)
+			(effects
+				(font
+					(size 1.27 1.27)
+				)
+				(hide yes)
+			)
+		)
+		(property "Datasheet" "~"
+			(at 24.13 152.4 0)
+			(effects
+				(font
+					(size 1.27 1.27)
+				)
+				(hide yes)
+			)
+		)
+		(property "Description" "Resistor"
+			(at 24.13 152.4 0)
+			(effects
+				(font
+					(size 1.27 1.27)
+				)
+				(hide yes)
+			)
+		)
+		(pin "1"
+		)
+		(pin "2"
+		)
+		(instances
+			(project "AEC_Speaker_Mic_System"
+				(path "/b4ee80b5-9d9a-4551-9b0c-6a8cb8d78ca3/b62903f4-3152-49f4-b9de-0aa5889c0444"
+					(reference "R54")
+					(unit 1)
+				)
+			)
+		)
+	)
+	(symbol
 		(lib_id "power:+5V")
 		(at 116.84 189.23 180)
@@
 				(path "/b4ee80b5-9d9a-4551-9b0c-6a8cb8d78ca3/b62903f4-3152-49f4-b9de-0aa5889c0444"
 					(reference "#PWR06")
+					(unit 1)
+				)
+			)
+		)
+	)
+	(symbol
+		(lib_id "power:+3.3V")
+		(at 17.78 152.4 0)
+		(unit 1)
+		(exclude_from_sim no)
+		(in_bom yes)
+		(on_board yes)
+		(dnp no)
+		(fields_autoplaced yes)
+		(property "Reference" "#PWR0417"
+			(at 17.78 156.21 0)
+			(effects
+				(font
+					(size 1.27 1.27)
+				)
+				(hide yes)
+			)
+		)
+		(property "Value" "+3.3V"
+			(at 17.78 147.32 0)
+			(effects
+				(font
+					(size 1.27 1.27)
+				)
+			)
+		)
+		(property "Footprint" ""
+			(at 17.78 152.4 0)
+			(effects
+				(font
+					(size 1.27 1.27)
+				)
+				(hide yes)
+			)
+		)
+		(property "Datasheet" ""
+			(at 17.78 152.4 0)
+			(effects
+				(font
+					(size 1.27 1.27)
+				)
+				(hide yes)
+			)
+		)
+		(property "Description" "Power symbol creates a global label with name \"+3.3V\""
+			(at 17.78 152.4 0)
+			(effects
+				(font
+					(size 1.27 1.27)
+				)
+				(hide yes)
+			)
+		)
+		(pin "1"
+		)
+		(instances
+			(project "AEC_Speaker_Mic_System"
+				(path "/b4ee80b5-9d9a-4551-9b0c-6a8cb8d78ca3/b62903f4-3152-49f4-b9de-0aa5889c0444"
+					(reference "#PWR0417")
 					(unit 1)
 				)
@@
 			(effects
 				(font
+					(size 1.27 1.27)
+				)
+				(justify left)
+			)
+		)
+		(pin "TACHOMETER" input
+			(at 203.2 149.86 180)
+			(effects
+				(font

Commit message: Fixed most ERC checks
Parts:
- renumbered C1 to C9, J1 to J2, J2 to J3, R54 to R5, R1 to R6, U1 to U3
Connections:
- no-connect marks 0 -> 60
Changed lines of the file:
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@@
 		(color 0 0 0 0)
+	)
+	(no_connect
+		(at 156.21 163.83)
+	)
+	(no_connect
+		(at 74.93 177.8)
+	)
+	(no_connect
+		(at 74.93 160.02)
+	)
+	(no_connect
+		(at 44.45 172.72)
+	)
+	(no_connect
+		(at 116.84 186.69)
+	)
+	(no_connect
+		(at 156.21 186.69)
+	)
+	(no_connect
+		(at 44.45 167.64)
+	)
+	(no_connect
+		(at 116.84 156.21)
+	)
+	(no_connect
+		(at 116.84 153.67)
+	)
+	(no_connect
+		(at 74.93 162.56)
+	)
+	(no_connect
+		(at 74.93 154.94)
+	)
+	(no_connect
+		(at 116.84 168.91)
+	)
+	(no_connect
+		(at 156.21 158.75)
+	)
+	(no_connect
+		(at 44.45 182.88)
+	)
+	(no_connect
+		(at 74.93 172.72)
+	)
+	(no_connect
+		(at 156.21 153.67)
+	)
+	(no_connect
+		(at 156.21 161.29)
+	)
+	(no_connect
+		(at 116.84 176.53)
+	)
+	(no_connect
+		(at 116.84 151.13)
+	)
+	(no_connect
+		(at 116.84 179.07)
+	)
+	(no_connect
+		(at 156.21 184.15)
+	)
+	(no_connect
+		(at 74.93 157.48)
+	)
+	(no_connect
+		(at 44.45 185.42)
+	)
+	(no_connect
+		(at 74.93 180.34)
+	)
+	(no_connect
+		(at 44.45 180.34)
+	)
+	(no_connect
+		(at 44.45 187.96)
+	)
+	(no_connect
+		(at 74.93 167.64)
+	)
+	(no_connect
+		(at 156.21 140.97)
+	)
+	(no_connect
+		(at 156.21 181.61)
+	)
+	(no_connect
+		(at 116.84 163.83)
+	)
+	(no_connect
+		(at 156.21 171.45)
+	)
+	(no_connect
+		(at 116.84 148.59)
+	)
+	(no_connect
+		(at 116.84 171.45)
+	)
+	(no_connect
+		(at 116.84 161.29)
+	)
+	(no_connect
+		(at 156.21 173.99)
+	)
+	(no_connect
+		(at 156.21 168.91)
+	)
+	(no_connect
+		(at 156.21 156.21)
+	)
+	(no_connect
+		(at 116.84 146.05)
+	)
+	(no_connect
+		(at 156.21 176.53)
+	)
+	(no_connect
+		(at 156.21 148.59)
+	)
+	(no_connect
+		(at 74.93 165.1)
+	)
+	(no_connect
+		(at 156.21 166.37)
+	)
+	(no_connect
+		(at 74.93 152.4)
+	)
+	(no_connect
+		(at 74.93 170.18)
+	)
+	(no_connect
+		(at 44.45 190.5)
+	)
+	(no_connect
+		(at 44.45 177.8)
+	)
+	(no_connect
+		(at 116.84 166.37)
+	)
+	(no_connect
+		(at 74.93 149.86)
+	)
+	(no_connect
+		(at 116.84 158.75)
+	)
+	(no_connect
+		(at 44.45 170.18)
+	)
+	(no_connect
+		(at 156.21 179.07)
+	)
+	(no_connect
+		(at 156.21 143.51)
+	)
+	(no_connect
+		(at 44.45 165.1)
+	)
+	(no_connect
+		(at 156.21 151.13)
+	)
+	(no_connect
+		(at 44.45 175.26)
+	)
+	(no_connect
+		(at 116.84 173.99)
+	)
+	(no_connect
+		(at 74.93 182.88)
+	)
+	(no_connect
+		(at 74.93 175.26)
+	)
+	(no_connect
+		(at 156.21 146.05)
+	)
+	(no_connect
+		(at 74.93 185.42)
 	)
 	(wire
@@
 		(dnp no)
 		(fields_autoplaced yes)
-		(property "Reference" "#PWR05"
+		(property "Reference" "#PWR024"
 			(at 43.18 137.16 0)
 			(effects
@@
 			(project "AEC_Speaker_Mic_System"
 				(path "/b4ee80b5-9d9a-4551-9b0c-6a8cb8d78ca3/b62903f4-3152-49f4-b9de-0aa5889c0444"
-					(reference "#PWR05")
+					(reference "#PWR024")
 					(unit 1)
 				)
@@
 		(on_board yes)
 		(dnp no)
-		(property "Reference" "C1"
+		(property "Reference" "C9"
 			(at 28.448 139.7 0)
 			(effects
@@
 			(project "AEC_Speaker_Mic_System"
 				(path "/b4ee80b5-9d9a-4551-9b0c-6a8cb8d78ca3/b62903f4-3152-49f4-b9de-0aa5889c0444"
-					(reference "C1")
+					(reference "C9")
 					(unit 1)
 				)
@@
 		(dnp no)
 		(fields_autoplaced yes)
-		(property "Reference" "#PWR01"
+		(property "Reference" "#PWR026"
 			(at 66.04 195.58 0)
 			(effects
@@
 			(project "AEC_Speaker_Mic_System"
 				(path "/b4ee80b5-9d9a-4551-9b0c-6a8cb8d78ca3/b62903f4-3152-49f4-b9de-0aa5889c0444"
-					(reference "#PWR01")
+					(reference "#PWR026")
 					(unit 1)
 				)
@@
 		(dnp no)
 		(fields_autoplaced yes)
-		(property "Reference" "#PWR04"
+		(property "Reference" "#PWR023"
 			(at 35.56 130.81 0)
 			(effects
@@
 			(project "AEC_Speaker_Mic_System"
 				(path "/b4ee80b5-9d9a-4551-9b0c-6a8cb8d78ca3/b62903f4-3152-49f4-b9de-0aa5889c0444"
-					(reference "#PWR04")
+					(reference "#PWR023")
 					(unit 1)
 				)
@@
 		(dnp no)
 		(fields_autoplaced yes)
-		(property "Reference" "U1"
+		(property "Reference" "U3"
 			(at 61.8333 137.16 0)
 			(effects
@@
 			(project "AEC_Speaker_Mic_System"
 				(path "/b4ee80b5-9d9a-4551-9b0c-6a8cb8d78ca3/b62903f4-3152-49f4-b9de-0aa5889c0444"
-					(reference "U1")
+					(reference "U3")
 					(unit 1)
 				)
@@
 		(dnp no)
 		(fields_autoplaced yes)
-		(property "Reference" "#PWR02"
+		(property "Reference" "#PWR025"
 			(at 50.8 143.51 0)
 			(effects
@@
 			(project "AEC_Speaker_Mic_System"
 				(path "/b4ee80b5-9d9a-4551-9b0c-6a8cb8d78ca3/b62903f4-3152-49f4-b9de-0aa5889c0444"
-					(reference "#PWR02")
+					(reference "#PWR025")
 					(unit 1)
 				)
@@
 		(dnp no)
 		(fields_autoplaced yes)
-		(property "Reference" "R54"
+		(property "Reference" "R5"
 			(at 24.13 146.05 90)
 			(effects
@@
 			(project "AEC_Speaker_Mic_System"
 				(path "/b4ee80b5-9d9a-4551-9b0c-6a8cb8d78ca3/b62903f4-3152-49f4-b9de-0aa5889c0444"
-					(reference "R54")
+					(reference "R5")
 					(unit 1)
 				)
@@
 		(on_board yes)
 		(dnp no)
-		(property "Reference" "#PWR06"
+		(property "Reference" "#PWR027"
 			(at 116.84 185.42 0)
 			(effects
@@
 			(project "AEC_Speaker_Mic_System"
 				(path "/b4ee80b5-9d9a-4551-9b0c-6a8cb8d78ca3/b62903f4-3152-49f4-b9de-0aa5889c0444"
-					(reference "#PWR06")
+					(reference "#PWR027")
 					(unit 1)
 				)
@@
 		(dnp no)
 		(fields_autoplaced yes)
-		(property "Reference" "#PWR0417"
+		(property "Reference" "#PWR022"
 			(at 17.78 156.21 0)
 			(effects
@@
 			(project "AEC_Speaker_Mic_System"
 				(path "/b4ee80b5-9d9a-4551-9b0c-6a8cb8d78ca3/b62903f4-3152-49f4-b9de-0aa5889c0444"
-					(reference "#PWR0417")
+					(reference "#PWR022")
 					(unit 1)
 				)
@@
 		(dnp no)
 		(fields_autoplaced yes)
-		(property "Reference" "J2"
+		(property "Reference" "J3"
 			(at 148.59 161.2901 0)
 			(effects
@@
 			(project "AEC_Speaker_Mic_System"
 				(path "/b4ee80b5-9d9a-4551-9b0c-6a8cb8d78ca3/b62903f4-3152-49f4-b9de-0aa5889c0444"
-					(reference "J2")
+					(reference "J3")
 					(unit 1)
 				)
@@
 		(on_board yes)
 		(dnp no)
-		(property "Reference" "J1"
+		(property "Reference" "J2"
 			(at 124.46 158.7499 0)
 			(effects
@@
 			(project "AEC_Speaker_Mic_System"
 				(path "/b4ee80b5-9d9a-4551-9b0c-6a8cb8d78ca3/b62903f4-3152-49f4-b9de-0aa5889c0444"
-					(reference "J1")
+					(reference "J2")
 					(unit 1)
 				)
@@
 		(dnp no)
 		(fields_autoplaced yes)
-		(property "Reference" "#PWR03"
+		(property "Reference" "#PWR028"
 			(at 162.56 189.23 0)
 			(effects
@@
 			(project "AEC_Speaker_Mic_System"
 				(path "/b4ee80b5-9d9a-4551-9b0c-6a8cb8d78ca3/b62903f4-3152-49f4-b9de-0aa5889c0444"
-					(reference "#PWR03")
+					(reference "#PWR028")
 					(unit 1)
 				)
@@
 		(dnp no)
 		(fields_autoplaced yes)
-		(property "Reference" "R1"
+		(property "Reference" "R6"
 			(at 45.72 135.8899 0)
 			(effects
@@
 			(project "AEC_Speaker_Mic_System"
 				(path "/b4ee80b5-9d9a-4551-9b0c-6a8cb8d78ca3/b62903f4-3152-49f4-b9de-0aa5889c0444"
-					(reference "R1")
+					(reference "R6")
 					(unit 1)
 				)
