File: _autosave-control_logic.kicad_sch (KiCad schematic)
At the start: 6 parts, among them J29 Cmod_A7_Right, J3 Cmod_A7_Left, U3 ESP32-S3-WROOM-1

Commit message: Cleared ERCs, need to footprint and switch THT for SMD
Parts:
- J29: symbol Cmod_A7_Right:Cmod_A7_Right -> Cmod_A7:Cmod_A7_Right
- J3: symbol Cmod_A7_Right:Cmod_A7_Left -> Cmod_A7:Cmod_A7_Left
Changed lines of the file:
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@@
 	)
 	(symbol
-		(lib_id "Cmod_A7_Right:Cmod_A7_Left")
+		(lib_id "Cmod_A7:Cmod_A7_Left")
 		(at 121.92 158.75 0)
 		(unit 1)
@@
 	)
 	(symbol
-		(lib_id "Cmod_A7_Right:Cmod_A7_Right")
+		(lib_id "Cmod_A7:Cmod_A7_Right")
 		(at 151.13 158.75 0)
 		(unit 1)
