File: AEC_Speaker_Mic_System.kicad_pcb (KiCad board)
At the start: 2 copper layers, 14.3 x 13.4 mm, 506 parts, among them CN1 XT60, J10 Screw_Terminal_01x02, J11 Screw_Terminal_01x02, J12 Screw_Terminal_01x02, J13 Screw_Terminal_01x02, J14 Screw_Terminal_01x02, J15 Screw_Terminal_01x02, J16 Conn_01x03_MountingPin, J19 Conn_01x03_MountingPin, J21 Conn_01x03_MountingPin, J23 Conn_01x03_MountingPin, J24 Conn_01x03_MountingPin, J26 Conn_01x03_MountingPin, J27 Conn_01x03_Pin, J29 Cmod_A7_Right, J3 Cmod_A7_Left, J8 Screw_Terminal_01x02, J9 Screw_Terminal_01x02, Q1 AO3400A, U1 AMS1117-3.3, U10 PCM5102A, U11 TPA3116D2DADR, U12 PCM5102A, U13 TPA3116D2DADR, U14 PCM5102A, U15 TPA3116D2DADR, U16 PCM5102A, U17 TPA3116D2DADR, U18 AP2112K-3.3TRG1, U19 AP2112K-1.8, U2 TPS62933, U20 TXB0104PW, U21 AP2112K-3.3TRG1, U22 AP2112K-1.8, U23 MAX3485, U24 MAX3485, U25 MAX3485, U26 MAX3485, U27 MAX3485, U28 MAX3485, U29 TXB0104PW, U3 ESP32-S3-WROOM-1, U30 AP2112K-3.3TRG1, U31 AP2112K-1.8, U32 MAX3485, U33 MAX3485, U34 MAX3485, U35 TXB0104PW, U36 AP2112K-3.3TRG1, U37 AP2112K-1.8, U38 MAX3485, U39 MAX3485, U4 MAX3485_SC, U40 MAX3485, U41 TXB0104PW, U42 TXB0104PW, U43 AP2112K-3.3TRG1, U44 AP2112K-1.8, U45 MAX3485, U46 MAX3485, U47 MAX3485, U48 TXB0104PW, U49 AP2112K-3.3TRG1, U5 MAX3485_WS, U50 AP2112K-1.8, U51 MAX3485, U52 LM393, U53 MAX3485, U54 MAX3485, U55 TPA3116D2DADR, U56 TPA3116D2DADR, U57 TPA3116D2DADR, U58 TPA3116D2DADR, U59 RJ45, U6 MAX3485_SD, U60 RJ45, U61 RJ45, U62 RJ45, U63 RJ45, U64 RJ45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

Commit message: Minor schematic changes
Parts:
- removed D6, D7: 1N4148W, Diode_SMD:D_SOD-123
- removed J19, J21, J23, J24, J26: Conn_01x03_MountingPin, Connector_PinHeader_2.54mm:PinHeader_1x03_P2.54mm_Vertical_SMD_Pin1Left
- removed J27: Conn_01x03_Pin, Connector_Molex:Molex_KK-254_AE-6410-03A_1x03_P2.54mm_Vertical
- removed J29: Cmod_A7_Right, Connector:HDR-TH_24P-P2.54-V-F-RIGHT_SIDE_NUMBERING
- added C289: 0.1u, Capacitor_SMD:C_0603_1608Metric, F.Cu at (77.6, 154.3)
- added C290: 0.1u, Capacitor_SMD:C_0603_1608Metric, F.Cu at (158.4, 125.6)
- added C291: 0.1u, Capacitor_SMD:C_0603_1608Metric, F.Cu at (77.6, 156.8)
- added C292: 0.1u, Capacitor_SMD:C_0603_1608Metric, F.Cu at (158.4, 128.1)
- added C293: 1u, Capacitor_SMD:C_0603_1608Metric, F.Cu at (152.4, 123.1)
- added C294: 2.2u, Capacitor_SMD:C_0603_1608Metric, F.Cu at (152.4, 125.6)
- added C295: 1u, Inductor_SMD:IND-SMD_L10.4-W10.3, F.Cu at (143.6, 127.8)
- added C296: 2.2u, Capacitor_SMD:C_0603_1608Metric, F.Cu at (152.4, 128.1)
- added C297: 10u, Capacitor_SMD:C_0603_1608Metric, F.Cu at (139.3, 92.7)
- added C298: 0.1u, Capacitor_SMD:C_0603_1608Metric, F.Cu at (158.4, 160.0)
- added C299: 0.1u, Capacitor_SMD:C_0603_1608Metric, F.Cu at (158.4, 162.5)
- added C300: 0.1u, Capacitor_SMD:C_0603_1608Metric, F.Cu at (158.4, 165.1)
- added C301: 1u, Capacitor_SMD:C_0603_1608Metric, F.Cu at (132.8, 141.7)
- added C302: 2.2u, Capacitor_SMD:C_0603_1608Metric, F.Cu at (132.8, 144.2)
- added C303: 1u, Inductor_SMD:IND-SMD_L10.4-W10.3, F.Cu at (123.9, 146.3)
- added C304: 2.2u, Capacitor_SMD:C_0603_1608Metric, F.Cu at (132.8, 146.7)
- added C305: 10u, Capacitor_SMD:C_0603_1608Metric, F.Cu at (107.9, 116.1)
- added C306: 0.1u, Capacitor_SMD:C_0603_1608Metric, F.Cu at (53.5, 151.8)
- added D1: D_Schottky, Diode_SMD:TO-277_3P-L5.4-W4.0-LS6.5-BR, F.Cu at (56.7, 95.9)
- added D2: SM4007, Diode_SMD:D_MELF, F.Cu at (68.5, 157.1)
- added J1: Cmod_A7_Left, Connector:HDR-TH_24P-P2.54-V-F, F.Cu at (31.0, 1.50)
- added J17: Conn_01x03_Pin, Connector_Molex:Molex_KK-254_AE-6410-03A_1x03_P2.54mm_Vertical, F.Cu at (57.8, 163.4)
- added J2: Cmod_A7_Right, Connector:HDR-TH_24P-P2.54-V-F-RIGHT_SIDE_NUMBERING, F.Cu at (29.7, 5.53)
- added J4: Screw_Terminal_01x02, TerminalBlock_Phoenix:CONN-TH_2P-P5.00_WJ500V-5.08-2P, F.Cu at (43.5, 120.0)
- added J5: Screw_Terminal_01x02, TerminalBlock_Phoenix:CONN-TH_2P-P5.00_WJ500V-5.08-2P, F.Cu at (43.5, 58.1)
- added J6: Screw_Terminal_01x02, TerminalBlock_Phoenix:CONN-TH_2P-P5.00_WJ500V-5.08-2P, F.Cu at (43.5, 69.7)
- added J7: Screw_Terminal_01x02, TerminalBlock_Phoenix:CONN-TH_2P-P5.00_WJ500V-5.08-2P, F.Cu at (108.5, 5.80)
- added R100: 10k, Resistor_SMD:R_0603_1608Metric, F.Cu at (53.5, 161.8)
- added R101: 120, Resistor_SMD:R_0603_1608Metric, F.Cu at (107.9, 118.6)
- C10, C9: value 0.1u -> 22u; footprint Capacitor_SMD:C_0603_1608Metric -> Capacitor_SMD:C_1206_3216Metric
- C100: value 0.22u -> 1u
- C101, C102: value 2.2u -> 220n
- C103, C104: value 0.68u -> 220n
- C105, C26, C78: value 0.68u -> 0.1u
- C106, C25, C27, C79, C80: value 0.68u -> 10u
- C107, C81: value 2.2n -> 10u
- C109, C157, C159, C165, C169, C188, C190, C192, C196, C202, C209, C39, C82, C83, C86: value 10u -> 0.1u
- C110: value 2.2n -> 100u
- C111, C171: value 10u -> 0.22u
- C112, C231, C232: value 1u -> 0.22u
- C113, C114, C115, C173, C174, C175, C234, C236: value 0.1u -> 0.68u
- C116, C233: value 1u -> 0.68u
- C117, C177, C178, C179, C180, C183, C239, C240, C244, C245, C246, C57, C59, C60, C65: value 10u -> 2n; footprint Capacitor_SMD:C_0603_1608Metric -> Capacitor_SMD:C_0805_2012Metric
- C118, C124, C184, C185, C186, C238, C63, C66: value 0.1u -> 2n; footprint Capacitor_SMD:C_0603_1608Metric -> Capacitor_SMD:C_0805_2012Metric
- C119, C243: value 100u -> 2n; footprint Capacitor_SMD:C_0603_1608Metric -> Capacitor_SMD:C_0805_2012Metric
- C120, C125, C237, C64: value 1u -> 2n; footprint Capacitor_SMD:C_0603_1608Metric -> Capacitor_SMD:C_0805_2012Metric
- C121, C131, C144, C24: value 2.2u -> 1u
- C122: value 1u -> 10u; footprint Inductor_SMD:IND-SMD_L10.4-W10.3 -> Capacitor_SMD:C_0603_1608Metric
- C123, C126: value 2.2u -> 2n; footprint Capacitor_SMD:C_0603_1608Metric -> Capacitor_SMD:C_0805_2012Metric
- C127: footprint Inductor_SMD:IND-SMD_L10.4-W10.3 -> Capacitor_SMD:C_0603_1608Metric
- C128, C136, C138, C142, C149, C23, C49, C72, C76: value 2.2u -> 0.1u
- C129, C134, C139, C140, C145, C189, C193, C195, C199, C242, C249, C253, C254, C255, C62: value 0.1u -> 10u
- C130, C146, C198, C206, C219: value 1u -> 0.1u
- C132, C143: value 1u -> 0.1u; footprint Inductor_SMD:IND-SMD_L10.4-W10.3 -> Capacitor_SMD:C_0603_1608Metric
- C133, C147, C20, C46, C75, C98: value 2.2u -> 10u
- C135, C141, C153, C205, C207, C218, C38: value 1u -> 10u
- C137: value 1u -> 100u; footprint Inductor_SMD:IND-SMD_L10.4-W10.3 -> Capacitor_SMD:C_0603_1608Metric
- C148: value 1u -> 2.2u; footprint Inductor_SMD:IND-SMD_L10.4-W10.3 -> Capacitor_SMD:C_0603_1608Metric
- C150, C151, C211, C90: value 1u -> 2.2u
- C152, C35: value 1u -> 2.2n
- C154: value 2200u -> 10u; footprint Capacitor_SMD:CAP-SMD_BD18.0-L19.0-W19.0-FD_EEEFK1E472SV -> Capacitor_SMD:C_0603_1608Metric
- C155: value 2200u -> 2.2n; footprint Capacitor_SMD:CAP-SMD_BD18.0-L19.0-W19.0-FD_EEEFK1E472SV -> Capacitor_SMD:C_0603_1608Metric
- C156, C181, C241, C247: value 10u -> 1u
- C16, C17, C18, C45, C68, C70, C97: value 220n -> 0.1u
- C160, C187, C191, C216, C251, C36, C40: value 0.1u -> 1u
- C161, C162, C163, C221, C223: value 0.1u -> 220n
- C164, C222: value 10u -> 220n
- C170: value 10u -> 100u
- C172: value 0.1u -> 0.22u
- C176, C235, C56: value 10u -> 0.68u
- C19, C69, C94: value 220n -> 10u
- C197: value 0.1u -> 100u
- C204, C67: value 100u -> 1u
- C208, C210, C88: value 0.1u -> 2.2u
- C21, C47, C48, C73, C74: value 0.22u -> 10u
- C212, C92: value 0.1u -> 2.2n
- C215: value 10u -> 2.2n
- C217: value 100u -> 0.1u
- C22, C99: value 0.22u -> 0.1u
- C224: value 1u -> 220n
- C256, C262, C263, C264, C271, C272, C273, C279, C280, C281, C287: value 2n -> 0.1u; footprint Capacitor_SMD:C_0805_2012Metric -> Capacitor_SMD:C_0603_1608Metric
- C257: value 2n -> 100u; footprint Capacitor_SMD:C_0805_2012Metric -> Capacitor_SMD:C_0603_1608Metric
- C258, C265, C274, C282: value 2n -> 1u; footprint Capacitor_SMD:C_0805_2012Metric -> Capacitor_SMD:C_0603_1608Metric
- C259, C261, C266, C268, C275, C277, C283, C285: value 2n -> 2.2u; footprint Capacitor_SMD:C_0805_2012Metric -> Capacitor_SMD:C_0603_1608Metric
- C260, C267, C276, C284: value 2n -> 1u; footprint Capacitor_SMD:C_0805_2012Metric -> Inductor_SMD:IND-SMD_L10.4-W10.3
- C269, C270, C278, C286: value 2n -> 10u; footprint Capacitor_SMD:C_0805_2012Metric -> Capacitor_SMD:C_0603_1608Metric
- C28: value 0.68u -> 2.2u
- C29: value 2.2n -> 0.1u
- C3, C6: value 0.1u -> 2200u; footprint Capacitor_SMD:C_0603_1608Metric -> Capacitor_SMD:CAP-SMD_BD18.0-L19.0-W19.0-FD_EEEFK1E472SV
- C30, C31, C91: value 10u -> 2.2u
- C4: value 10u -> 0.1u; footprint Capacitor_SMD:C_1210_3225Metric -> Capacitor_SMD:C_0603_1608Metric
- C41: value 100u -> 220n
- C5: value 10n -> 10u; footprint Capacitor_SMD:C_0603_1608Metric -> Capacitor_SMD:C_1210_3225Metric
- C50: value 2.2u -> 100u
- C51, C52: value 0.68u -> 0.22u
- C55: value 2.2n -> 0.68u
- C58: value 2.2n -> 2n; footprint Capacitor_SMD:C_0603_1608Metric -> Capacitor_SMD:C_0805_2012Metric
- C7: value 22u -> 10n; footprint Capacitor_SMD:C_1206_3216Metric -> Capacitor_SMD:C_0603_1608Metric
- C71, C96: value 220n -> 1u
- C77: value 0.68u -> 100u
- C8: value 22u -> 0.1u; footprint Capacitor_SMD:C_1206_3216Metric -> Capacitor_SMD:C_0603_1608Metric
- C84: value 2.2n -> 1u
- C93: value 100u -> 10u
- C95: value 220n -> 2.2n
- D4: value D_Schottky -> 1N4148W; footprint Diode_SMD:TO-277_3P-L5.4-W4.0-LS6.5-BR -> Diode_SMD:D_SOD-123
- D5: value SM4007 -> 1N4148W; footprint Diode_SMD:D_MELF -> Diode_SMD:D_SOD-123
- J11, J12, J13, J14, J15: value Screw_Terminal_01x02 -> Conn_01x03_MountingPin; footprint TerminalBlock_Phoenix:CONN-TH_2P-P5.00_WJ500V-5.08-2P -> Connector_PinHeader_2.54mm:PinHeader_1x03_P2.54mm_Vertical_SMD_Pin1Left
- J3: value Cmod_A7_Left -> Screw_Terminal_01x02; footprint Connector:HDR-TH_24P-P2.54-V-F -> TerminalBlock_Phoenix:CONN-TH_2P-P5.00_WJ500V-5.08-2P
- R10: value 120 -> 10; footprint Resistor_SMD:R_0603_1608Metric -> Resistor_SMD:R_0805_2012Metric
- R11, R19, R27, R32, R37, R63, R75, R96, R97: value 10 -> 100k; footprint Resistor_SMD:R_0805_2012Metric -> Resistor_SMD:R_0603_1608Metric
- R12, R30: value 10 -> 75k; footprint Resistor_SMD:R_0805_2012Metric -> Resistor_SMD:R_0603_1608Metric
- R13, R23, R67: value 10 -> 47k; footprint Resistor_SMD:R_0805_2012Metric -> Resistor_SMD:R_0603_1608Metric
- R14, R21, R29: value 470 -> 100k
- R15, R28, R35, R36: value 470 -> 10; footprint Resistor_SMD:R_0603_1608Metric -> Resistor_SMD:R_0805_2012Metric
- R17, R38, R46, R51, R52, R70, R74: value 100k -> 10; footprint Resistor_SMD:R_0603_1608Metric -> Resistor_SMD:R_0805_2012Metric
- R2: value 42.3k -> 43.2k
- R22: value 470 -> 75k
- R25, R26: value 10 -> 470; footprint Resistor_SMD:R_0805_2012Metric -> Resistor_SMD:R_0603_1608Metric
- R31, R41, R49: value 100k -> 47k
- R40, R48: value 10k -> 75k
- R42, R47, R50: value 10k -> 100k
- R43: value 100k -> 470
- R44: value 10k -> 470
- R54: value 10k -> 10; footprint Resistor_SMD:R_0603_1608Metric -> Resistor_SMD:R_0805_2012Metric
- R55, R57, R68: value 75k -> 100k
- R56, R64, R72: value 75k -> 10; footprint Resistor_SMD:R_0603_1608Metric -> Resistor_SMD:R_0805_2012Metric
- R60, R65, R73: value 47k -> 100k
- R61, R62: value 47k -> 470
- R66: value 100k -> 75k
- R69: value 47k -> 10; footprint Resistor_SMD:R_0603_1608Metric -> Resistor_SMD:R_0805_2012Metric
- R7, R8: value 120 -> 470
- R80, R84, R87, R91, R92: value 100k -> 10k
- R81, R83, R85, R88, R93: value 100k -> 120
- R9: value 120 -> 100k
- R95: value 10 -> 10k; footprint Resistor_SMD:R_0805_2012Metric -> Resistor_SMD:R_0603_1608Metric
- U10, U12: value PCM5102A -> RJ45; footprint Package_SO:TSSOP-20_4.4x6.5mm_P0.65mm -> Connector:RJ45-SMD_HC-RJ45-055-4_2
- U11, U13: value TPA3116D2DADR -> MAX3485_SD; footprint TPA3116D2DADR:SOP65P810X115-33N -> Package_SO:SOIC-8_3.9x4.9mm_P1.27mm
- U16: value PCM5102A -> TPA3116D2DADR; footprint Package_SO:TSSOP-20_4.4x6.5mm_P0.65mm -> TPA3116D2DADR:SOP65P810X115-33N
- U17: value TPA3116D2DADR -> PCM5102A; footprint TPA3116D2DADR:SOP65P810X115-33N -> Package_SO:TSSOP-20_4.4x6.5mm_P0.65mm
- U18, U21: value AP2112K-3.3TRG1 -> TPA3116D2DADR; footprint AP2112K-3.3TRG1:SOT95P285X140-5N -> TPA3116D2DADR:SOP65P810X115-33N
- U19, U22: value AP2112K-1.8 -> TPA3116D2DADR; footprint Package_TO_SOT_SMD:SOT-23-5 -> TPA3116D2DADR:SOP65P810X115-33N
- U20: value TXB0104PW -> PCM5102A; footprint Package_SO:TSSOP-14_4.4x5mm_P0.65mm -> Package_SO:TSSOP-20_4.4x6.5mm_P0.65mm
- U23: value MAX3485 -> PCM5102A; footprint Package_SO:SOIC-8_3.9x4.9mm_P1.27mm -> Package_SO:TSSOP-20_4.4x6.5mm_P0.65mm
- U24, U25: value MAX3485 -> TPA3116D2DADR; footprint Package_SO:SOIC-8_3.9x4.9mm_P1.27mm -> TPA3116D2DADR:SOP65P810X115-33N
- U26, U40, U47: value MAX3485 -> AP2112K-3.3TRG1; footprint Package_SO:SOIC-8_3.9x4.9mm_P1.27mm -> AP2112K-3.3TRG1:SOT95P285X140-5N
- U27: value MAX3485 -> AP2112K-1.8; footprint Package_SO:SOIC-8_3.9x4.9mm_P1.27mm -> Package_TO_SOT_SMD:SOT-23-5
- U28, U39, U46, U53, U54: value MAX3485 -> TXB0104PW; footprint Package_SO:SOIC-8_3.9x4.9mm_P1.27mm -> Package_SO:TSSOP-14_4.4x5mm_P0.65mm
- U29: value TXB0104PW -> AP2112K-3.3TRG1; footprint Package_SO:TSSOP-14_4.4x5mm_P0.65mm -> AP2112K-3.3TRG1:SOT95P285X140-5N
- U30: value AP2112K-3.3TRG1 -> AP2112K-1.8; footprint AP2112K-3.3TRG1:SOT95P285X140-5N -> Package_TO_SOT_SMD:SOT-23-5
- U31, U37, U44: value AP2112K-1.8 -> MAX3485; footprint Package_TO_SOT_SMD:SOT-23-5 -> Package_SO:SOIC-8_3.9x4.9mm_P1.27mm
- U32: value MAX3485 -> RJ45; footprint Package_SO:SOIC-8_3.9x4.9mm_P1.27mm -> Connector:RJ45-SMD_HC-RJ45-055-4_2
- U35, U42: value TXB0104PW -> MAX3485; footprint Package_SO:TSSOP-14_4.4x5mm_P0.65mm -> Package_SO:SOIC-8_3.9x4.9mm_P1.27mm
- U36, U43: value AP2112K-3.3TRG1 -> RJ45; footprint AP2112K-3.3TRG1:SOT95P285X140-5N -> Connector:RJ45-SMD_HC-RJ45-055-4_2
- U41, U48: value TXB0104PW -> AP2112K-1.8; footprint Package_SO:TSSOP-14_4.4x5mm_P0.65mm -> Package_TO_SOT_SMD:SOT-23-5
- U49: value AP2112K-3.3TRG1 -> MAX3485; footprint AP2112K-3.3TRG1:SOT95P285X140-5N -> Package_SO:SOIC-8_3.9x4.9mm_P1.27mm
- U50: value AP2112K-1.8 -> RJ45; footprint Package_TO_SOT_SMD:SOT-23-5 -> Connector:RJ45-SMD_HC-RJ45-055-4_2
- U52: value LM393 -> MAX3485
- U55: value TPA3116D2DADR -> AP2112K-3.3TRG1; footprint TPA3116D2DADR:SOP65P810X115-33N -> AP2112K-3.3TRG1:SOT95P285X140-5N
- U56: value TPA3116D2DADR -> AP2112K-1.8; footprint TPA3116D2DADR:SOP65P810X115-33N -> Package_TO_SOT_SMD:SOT-23-5
- U57: value TPA3116D2DADR -> MAX3485; footprint TPA3116D2DADR:SOP65P810X115-33N -> Package_SO:SOIC-8_3.9x4.9mm_P1.27mm
- U58: value TPA3116D2DADR -> RJ45; footprint TPA3116D2DADR:SOP65P810X115-33N -> Connector:RJ45-SMD_HC-RJ45-055-4_2
- U59, U60, U64, U67, U68: value RJ45 -> MAX3485; footprint Connector:RJ45-SMD_HC-RJ45-055-4_2 -> Package_SO:SOIC-8_3.9x4.9mm_P1.27mm
- U6, U8: value MAX3485_SD -> RJ45; footprint Package_SO:SOIC-8_3.9x4.9mm_P1.27mm -> Connector:RJ45-SMD_HC-RJ45-055-4_2
- U61: value RJ45 -> TXB0104PW; footprint Connector:RJ45-SMD_HC-RJ45-055-4_2 -> Package_SO:TSSOP-14_4.4x5mm_P0.65mm
- U62: value RJ45 -> AP2112K-3.3TRG1; footprint Connector:RJ45-SMD_HC-RJ45-055-4_2 -> AP2112K-3.3TRG1:SOT95P285X140-5N
- U63: value RJ45 -> AP2112K-1.8; footprint Connector:RJ45-SMD_HC-RJ45-055-4_2 -> Package_TO_SOT_SMD:SOT-23-5
- U66: value RJ45 -> LM393; footprint Connector:RJ45-SMD_HC-RJ45-055-4_2 -> Package_SO:SOIC-8_3.9x4.9mm_P1.27mm
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Connections:
- C10 pad 1: GND -> +5V
- C10 pad 2: +3.3V -> GND
- C100 pad 1: /PCB_Control/Amp_Control_Module_78/SPK_L_P -> GND
- C100 pad 2: /PCB_Control/Amp_Control_Module_78/SPK_L_N -> +24V
- C101 pad 1: GND -> /PCB_Control/Amp_Control_Module_34/W_BSPR
- C101 pad 2: Net-(U16-LDOO) -> /PCB_Control/Amp_Control_Module_34/W_OUTPR
- C102 pad 1: GND -> /PCB_Control/Amp_Control_Module_34/W_BSNR
- C102 pad 2: Net-(U16-VNEG) -> /PCB_Control/Amp_Control_Module_34/W_OUTNR
- C103 pad 1: GND -> /PCB_Control/Amp_Control_Module_34/W_BSPL
- C103 pad 2: /PCB_Control/Amp_Control_Module_78/SPK_R_P -> /PCB_Control/Amp_Control_Module_34/W_OUTPL
- C104 pad 1: GND -> /PCB_Control/Amp_Control_Module_34/W_BSNL
- C104 pad 2: /PCB_Control/Amp_Control_Module_78/SPK_L_P -> /PCB_Control/Amp_Control_Module_34/W_OUTNL
- C105 pad 2: /PCB_Control/Amp_Control_Module_78/SPK_R_N -> +24V
- C106 pad 2: /PCB_Control/Amp_Control_Module_78/SPK_L_N -> +24V
- C107 pad 1: Net-(C107-Pad1) -> GND
- C107 pad 2: GND -> +24V
- C108 pad 1: Net-(C107-Pad1) -> GND
- C108 pad 2: /PCB_Control/Amp_Control_Module_78/LEFT_INPUT -> +24V
- C109 pad 1: Net-(C109-Pad1) -> GND
- C109 pad 2: /PCB_Control/Amp_Control_Module_78/RIGHT_INPUT -> +24V
- C11 pad 2: +3.3V -> Net-(U3-EN)
- C110 pad 1: Net-(C109-Pad1) -> GND
- C110 pad 2: GND -> +24V
- C111 pad 1: GND -> /PCB_Control/Amp_Control_Module_34/SPK_R_P
- C111 pad 2: Net-(U17-LINN) -> /PCB_Control/Amp_Control_Module_34/SPK_R_N
- C112 pad 1: Net-(U56-GVDD) -> /PCB_Control/Amp_Control_Module_34/SPK_L_P
- C112 pad 2: GND -> /PCB_Control/Amp_Control_Module_34/SPK_L_N
- C113 pad 2: +24V -> /PCB_Control/Amp_Control_Module_34/SPK_R_P
- C114 pad 2: +24V -> /PCB_Control/Amp_Control_Module_34/SPK_L_P
- C115 pad 2: +24V -> /PCB_Control/Amp_Control_Module_34/SPK_R_N
- C116 pad 2: +24V -> /PCB_Control/Amp_Control_Module_34/SPK_L_N
- C117 pad 1: GND -> /PCB_Control/Amp_Control_Module_34/SPK_R_P
- C117 pad 2: +24V -> GND
- C118 pad 2: +24V -> /PCB_Control/Amp_Control_Module_34/SPK_R_N
- C119 pad 1: GND -> /PCB_Control/Amp_Control_Module_34/SPK_L_P
- C119 pad 2: +24V -> GND
- C120 pad 1: /Breakout_1/+5V_CABLE -> GND
- C120 pad 2: /Breakout_1/GND_LOCAL -> /PCB_Control/Amp_Control_Module_34/SPK_L_N
- C121 pad 1: /Breakout_1/GND_LOCAL -> /PCB_Control/Amp_Control_Module_34/VD_PLIMIT_R
- C121 pad 2: /Breakout_1/+3.3V_LOCAL -> GND
- C122 pad 1: /Breakout_1/+5V_CABLE -> GND
- C122 pad 2: /Breakout_1/GND_LOCAL -> Net-(U19-LINN)
- C123 pad 1: /Breakout_1/GND_LOCAL -> Net-(C123-Pad1)
- C123 pad 2: /Breakout_1/+1V8_LOCAL -> GND
- C124 pad 1: /Breakout_4/+1V8_LOCAL -> Net-(C124-Pad1)
- C124 pad 2: /Breakout_4/GND_LOCAL -> GND
- C125 pad 1: /Breakout_4/+5V_CABLE -> Net-(C125-Pad1)
- C125 pad 2: /Breakout_4/GND_LOCAL -> GND
- C126 pad 1: /Breakout_4/GND_LOCAL -> Net-(C126-Pad1)
- C126 pad 2: /Breakout_4/+3.3V_LOCAL -> GND
- C127 pad 1: /Breakout_4/+5V_CABLE -> Net-(U19-GVDD)
- C127 pad 2: /Breakout_4/GND_LOCAL -> GND
- C128 pad 1: /Breakout_4/GND_LOCAL -> GND
- C128 pad 2: /Breakout_4/+1V8_LOCAL -> +24V
- C129 pad 1: /Breakout_2/+1V8_LOCAL -> GND
- C129 pad 2: /Breakout_2/GND_LOCAL -> +24V
- C130 pad 1: /Breakout_2/+5V_CABLE -> GND
- C130 pad 2: /Breakout_2/GND_LOCAL -> +24V
- C131 pad 1: /Breakout_2/GND_LOCAL -> GND
- C131 pad 2: /Breakout_2/+3.3V_LOCAL -> +24V
- C132 pad 1: /Breakout_2/+5V_CABLE -> GND
- C132 pad 2: /Breakout_2/GND_LOCAL -> +24V
- C133 pad 1: /Breakout_2/GND_LOCAL -> GND
- C133 pad 2: /Breakout_2/+1V8_LOCAL -> +24V
- C134 pad 1: /Breakout_5/+1V8_LOCAL -> GND
- C134 pad 2: /Breakout_5/GND_LOCAL -> +24V
- C135 pad 1: /Breakout_5/+5V_CABLE -> GND
- C135 pad 2: /Breakout_5/GND_LOCAL -> +24V
- C136 pad 1: /Breakout_5/GND_LOCAL -> GND
- C136 pad 2: /Breakout_5/+3.3V_LOCAL -> +24V
- C137 pad 1: /Breakout_5/+5V_CABLE -> GND
- C137 pad 2: /Breakout_5/GND_LOCAL -> +24V
- C138 pad 1: /Breakout_5/GND_LOCAL -> GND
- C138 pad 2: /Breakout_5/+1V8_LOCAL -> +3.3V
- C139 pad 1: /Breakout_3/+1V8_LOCAL -> GND
- C139 pad 2: /Breakout_3/GND_LOCAL -> +3.3V
- C140 pad 1: /Breakout_1/+1V8_LOCAL -> GND
- C140 pad 2: /Breakout_1/GND_LOCAL -> +3.3V
- C141 pad 1: /Breakout_3/+5V_CABLE -> GND
- C141 pad 2: /Breakout_3/GND_LOCAL -> GND
- C142 pad 1: /Breakout_3/GND_LOCAL -> GND
- C142 pad 2: /Breakout_3/+3.3V_LOCAL -> +3.3V
- C143 pad 1: /Breakout_3/+5V_CABLE -> GND
- C143 pad 2: /Breakout_3/GND_LOCAL -> GND
- C144 pad 1: /Breakout_3/GND_LOCAL -> /PCB_Control/Amp_Control_Module_56/VD_PLIMIT_L
- C144 pad 2: /Breakout_3/+1V8_LOCAL -> GND
- C145 pad 1: /Breakout_6/+1V8_LOCAL -> GND
- C145 pad 2: /Breakout_6/GND_LOCAL -> Net-(U21-LINN)
- C146 pad 1: /Breakout_6/+5V_CABLE -> GND
- C146 pad 2: /Breakout_6/GND_LOCAL -> GND
- C147 pad 1: /Breakout_6/GND_LOCAL -> GND
- C147 pad 2: /Breakout_6/+3.3V_LOCAL -> +3.3V
- C148 pad 1: /Breakout_6/+5V_CABLE -> Net-(U20-CAPP)
- C148 pad 2: /Breakout_6/GND_LOCAL -> Net-(U20-CAPM)
- C149 pad 1: /Breakout_6/GND_LOCAL -> GND
- C149 pad 2: /Breakout_6/+1V8_LOCAL -> +3.3V
- C150 pad 1: /PCB_Control/Amp_Control_Module_12/VD_PLIMIT_L -> GND
- C150 pad 2: GND -> Net-(U20-LDOO)
- C151 pad 1: /PCB_Control/Amp_Control_Module_34/VD_PLIMIT_L -> GND
- C151 pad 2: GND -> Net-(U20-VNEG)
- C152 pad 1: /PCB_Control/Amp_Control_Module_56/VD_PLIMIT_L -> Net-(C152-Pad1)
- C153 pad 1: /PCB_Control/Amp_Control_Module_78/VD_PLIMIT_L -> Net-(C152-Pad1)
- C153 pad 2: GND -> /PCB_Control/Amp_Control_Module_56/LEFT_INPUT
- C154 pad 1: +24V -> Net-(C154-Pad1)
- C154 pad 2: GND -> /PCB_Control/Amp_Control_Module_56/RIGHT_INPUT
- C155 pad 1: +24V -> Net-(C154-Pad1)
- C156 pad 1: GND -> Net-(U21-GVDD)
- C156 pad 2: +24V -> GND
- C16 pad 1: /PCB_Control/Amp_Control_Module_12/W_BSPR -> GND
- C16 pad 2: /PCB_Control/Amp_Control_Module_12/W_OUTPR -> +3.3V
- C161 pad 1: GND -> /PCB_Control/Amp_Control_Module_56/W_BSPR
- C161 pad 2: +24V -> /PCB_Control/Amp_Control_Module_56/W_OUTPR
- C162 pad 1: GND -> /PCB_Control/Amp_Control_Module_56/W_BSNR
- C162 pad 2: +24V -> /PCB_Control/Amp_Control_Module_56/W_OUTNR
- C163 pad 1: GND -> /PCB_Control/Amp_Control_Module_56/W_BSPL
- C163 pad 2: +24V -> /PCB_Control/Amp_Control_Module_56/W_OUTPL
- C164 pad 1: GND -> /PCB_Control/Amp_Control_Module_56/W_BSNL
- C164 pad 2: +24V -> /PCB_Control/Amp_Control_Module_56/W_OUTNL
- C17 pad 1: /PCB_Control/Amp_Control_Module_12/W_BSNR -> GND
- C17 pad 2: /PCB_Control/Amp_Control_Module_12/W_OUTNR -> +3.3V
- C171 pad 1: GND -> /PCB_Control/Amp_Control_Module_56/SPK_R_P
- C171 pad 2: +24V -> /PCB_Control/Amp_Control_Module_56/SPK_R_N
- C172 pad 1: GND -> /PCB_Control/Amp_Control_Module_56/SPK_L_P
- C172 pad 2: +3.3V -> /PCB_Control/Amp_Control_Module_56/SPK_L_N
- C173 pad 2: +3.3V -> /PCB_Control/Amp_Control_Module_56/SPK_R_P
- C174 pad 2: +3.3V -> /PCB_Control/Amp_Control_Module_56/SPK_L_P
- C175 pad 2: +3.3V -> /PCB_Control/Amp_Control_Module_56/SPK_R_N
- C176 pad 2: +3.3V -> /PCB_Control/Amp_Control_Module_56/SPK_L_N
- C177 pad 1: GND -> /PCB_Control/Amp_Control_Module_56/SPK_R_P
- C177 pad 2: +3.3V -> GND
- C178 pad 2: +3.3V -> /PCB_Control/Amp_Control_Module_56/SPK_R_N
- C179 pad 1: GND -> /PCB_Control/Amp_Control_Module_56/SPK_L_P
- C179 pad 2: +3.3V -> GND
- C18 pad 1: /PCB_Control/Amp_Control_Module_12/W_BSPL -> GND
- C18 pad 2: /PCB_Control/Amp_Control_Module_12/W_OUTPL -> +3.3V
- C180 pad 2: +3.3V -> /PCB_Control/Amp_Control_Module_56/SPK_L_N
- C181 pad 1: GND -> /PCB_Control/Amp_Control_Module_56/VD_PLIMIT_R
- C181 pad 2: +3.3V -> GND
- C182 pad 2: +3.3V -> Net-(U22-LINN)
- C183 pad 1: GND -> Net-(C183-Pad1)
- C183 pad 2: +3.3V -> GND
- C184 pad 1: GND -> Net-(C184-Pad1)
- C184 pad 2: +3.3V -> GND
- C185 pad 1: GND -> Net-(C185-Pad1)
- C185 pad 2: +3.3V -> GND
- C186 pad 1: GND -> Net-(C186-Pad1)
- C186 pad 2: +3.3V -> GND
- C187 pad 1: GND -> Net-(U22-GVDD)
- C187 pad 2: +3.3V -> GND
- C188 pad 2: +3.3V -> +24V
- C189 pad 2: +3.3V -> +24V
- C19 pad 1: /PCB_Control/Amp_Control_Module_12/W_BSNL -> GND
- C19 pad 2: /PCB_Control/Amp_Control_Module_12/W_OUTNL -> +3.3V
- C190 pad 2: +3.3V -> +24V
- C191 pad 2: +3.3V -> +24V
- C192 pad 2: +3.3V -> +24V
- C193 pad 2: +3.3V -> +24V
- C194 pad 2: +3.3V -> +24V
- C195 pad 2: +3.3V -> +24V
- C198 pad 2: +24V -> +3.3V
- C199 pad 2: +24V -> +3.3V
- C20 pad 1: Net-(U10-CAPP) -> GND
- C20 pad 2: Net-(U10-CAPM) -> +3.3V
- C200 pad 2: +24V -> +3.3V
- C201 pad 2: +24V -> GND
- C202 pad 2: +24V -> +3.3V
- C203 pad 2: +24V -> GND
- C204 pad 1: GND -> /PCB_Control/Amp_Control_Module_78/VD_PLIMIT_L
- C204 pad 2: +24V -> GND
- C205 pad 1: /PCB_Control/Amp_Control_Module_34/VD_PLIMIT_R -> GND
- C205 pad 2: GND -> Net-(U24-LINN)
- C206 pad 1: Net-(U57-GVDD) -> GND
- C207 pad 1: Net-(U58-GVDD) -> GND
- C207 pad 2: GND -> +3.3V
- C208 pad 1: GND -> Net-(U23-CAPP)
- C208 pad 2: +24V -> Net-(U23-CAPM)
- C209 pad 2: +24V -> +3.3V
- C21 pad 1: /PCB_Control/Amp_Control_Module_12/SPK_R_P -> GND
- C21 pad 2: /PCB_Control/Amp_Control_Module_12/SPK_R_N -> GND
- C210 pad 2: +24V -> Net-(U23-LDOO)
- C211 pad 2: +24V -> Net-(U23-VNEG)
- C212 pad 1: GND -> Net-(C212-Pad1)
- C212 pad 2: +24V -> GND
- C213 pad 1: GND -> Net-(C212-Pad1)
- C213 pad 2: +24V -> /PCB_Control/Amp_Control_Module_78/LEFT_INPUT
- C214 pad 1: GND -> Net-(C214-Pad1)
- C214 pad 2: +24V -> /PCB_Control/Amp_Control_Module_78/RIGHT_INPUT
- C215 pad 1: GND -> Net-(C214-Pad1)
- C215 pad 2: +24V -> GND
- C216 pad 1: GND -> Net-(U24-GVDD)
- C216 pad 2: +24V -> GND
- C218 pad 1: /PCB_Control/Amp_Control_Module_56/VD_PLIMIT_R -> GND
- C218 pad 2: GND -> +24V
- C219 pad 1: Net-(U11-GVDD) -> GND
- C219 pad 2: GND -> +24V
- C22 pad 1: /PCB_Control/Amp_Control_Module_12/SPK_L_P -> GND
- C22 pad 2: /PCB_Control/Amp_Control_Module_12/SPK_L_N -> +3.3V
- C220 pad 1: Net-(U13-GVDD) -> GND
- C220 pad 2: GND -> +24V
- C221 pad 1: GND -> /PCB_Control/Amp_Control_Module_78/W_BSPR
- C221 pad 2: +24V -> /PCB_Control/Amp_Control_Module_78/W_OUTPR
- C222 pad 1: GND -> /PCB_Control/Amp_Control_Module_78/W_BSNR
- C222 pad 2: +24V -> /PCB_Control/Amp_Control_Module_78/W_OUTNR
- C223 pad 1: GND -> /PCB_Control/Amp_Control_Module_78/W_BSPL
- C223 pad 2: +24V -> /PCB_Control/Amp_Control_Module_78/W_OUTPL
- C224 pad 1: GND -> /PCB_Control/Amp_Control_Module_78/W_BSNL
- C224 pad 2: +24V -> /PCB_Control/Amp_Control_Module_78/W_OUTNL
- C23 pad 2: Net-(U10-LDOO) -> GND
- C231 pad 1: /PCB_Control/Amp_Control_Module_78/VD_PLIMIT_R -> /PCB_Control/Amp_Control_Module_78/SPK_R_P
- C231 pad 2: GND -> /PCB_Control/Amp_Control_Module_78/SPK_R_N
- C232 pad 1: Net-(U15-GVDD) -> /PCB_Control/Amp_Control_Module_78/SPK_L_P
- C232 pad 2: GND -> /PCB_Control/Amp_Control_Module_78/SPK_L_N
- C233 pad 1: Net-(U17-GVDD) -> GND
- C233 pad 2: GND -> /PCB_Control/Amp_Control_Module_78/SPK_R_P
- C234 pad 2: +24V -> /PCB_Control/Amp_Control_Module_78/SPK_L_P
- C235 pad 2: +24V -> /PCB_Control/Amp_Control_Module_78/SPK_R_N
- C236 pad 2: +24V -> /PCB_Control/Amp_Control_Module_78/SPK_L_N
- C237 pad 1: GND -> /PCB_Control/Amp_Control_Module_78/SPK_R_P
- C237 pad 2: +24V -> GND
- C238 pad 2: +24V -> /PCB_Control/Amp_Control_Module_78/SPK_R_N
- C239 pad 1: GND -> /PCB_Control/Amp_Control_Module_78/SPK_L_P
- C239 pad 2: +24V -> GND
- C24 pad 1: GND -> /PCB_Control/Amp_Control_Module_12/VD_PLIMIT_L
- C24 pad 2: Net-(U10-VNEG) -> GND
- C240 pad 2: +24V -> /PCB_Control/Amp_Control_Module_78/SPK_L_N
- C241 pad 1: GND -> /PCB_Control/Amp_Control_Module_78/VD_PLIMIT_R
- C241 pad 2: +24V -> GND
- C242 pad 2: +24V -> Net-(U25-LINN)
- C243 pad 1: GND -> Net-(C243-Pad1)
- C243 pad 2: +24V -> GND
- C244 pad 1: GND -> Net-(C244-Pad1)
- C245 pad 1: GND -> Net-(C245-Pad1)
- C246 pad 1: GND -> Net-(C246-Pad1)
- C247 pad 1: GND -> Net-(U25-GVDD)
- C248 pad 2: GND -> +24V
- C249 pad 2: GND -> +24V
- C25 pad 2: /PCB_Control/Amp_Control_Module_12/SPK_R_P -> Net-(U15-LINN)
- C250 pad 2: GND -> +24V
- C251 pad 2: GND -> +24V
- C252 pad 2: GND -> +24V
- C253 pad 2: GND -> +24V
- C254 pad 2: GND -> +24V
- C255 pad 2: GND -> +24V
- C256 pad 2: /PCB_Control/Amp_Control_Module_12/SPK_L_N -> +24V
- C257 pad 2: /PCB_Control/Amp_Control_Module_34/SPK_L_N -> +24V
- C258 pad 1: GND -> /Breakout_1/+5V_CABLE
- C258 pad 2: /PCB_Control/Amp_Control_Module_56/SPK_L_N -> /Breakout_1/GND_LOCAL
- C259 pad 1: GND -> /Breakout_1/GND_LOCAL
- C259 pad 2: /PCB_Control/Amp_Control_Module_78/SPK_L_N -> /Breakout_1/+3.3V_LOCAL
- C26 pad 2: /PCB_Control/Amp_Control_Module_12/SPK_L_P -> GND
- C260 pad 1: /PCB_Control/Amp_Control_Module_12/SPK_L_P -> /Breakout_1/+5V_CABLE
- C260 pad 2: GND -> /Breakout_1/GND_LOCAL
- C261 pad 1: /PCB_Control/Amp_Control_Module_34/SPK_L_P -> /Breakout_1/GND_LOCAL
- C261 pad 2: GND -> /Breakout_1/+1V8_LOCAL
- C262 pad 1: /PCB_Control/Amp_Control_Module_56/SPK_L_P -> /Breakout_4/+1V8_LOCAL
- C262 pad 2: GND -> /Breakout_4/GND_LOCAL
- C263 pad 1: /PCB_Control/Amp_Control_Module_78/SPK_L_P -> /Breakout_4/GND_LOCAL
- C263 pad 2: GND -> /Breakout_4/+1V8_LOCAL
- C264 pad 1: Net-(C264-Pad1) -> /Breakout_4/+3.3V_LOCAL
- C264 pad 2: GND -> /Breakout_4/GND_LOCAL
- C265 pad 1: Net-(C265-Pad1) -> /Breakout_4/+5V_CABLE
- C265 pad 2: GND -> /Breakout_4/GND_LOCAL
- C266 pad 1: Net-(C266-Pad1) -> /Breakout_4/GND_LOCAL
- C266 pad 2: GND -> /Breakout_4/+3.3V_LOCAL
- C267 pad 1: Net-(C267-Pad1) -> /Breakout_4/+5V_CABLE
- C267 pad 2: GND -> /Breakout_4/GND_LOCAL
- C268 pad 1: Net-(C268-Pad1) -> /Breakout_4/GND_LOCAL
- C268 pad 2: GND -> /Breakout_4/+1V8_LOCAL
- C269 pad 1: Net-(C269-Pad1) -> /Breakout_4/GND_LOCAL
- C269 pad 2: GND -> /Breakout_4/+5V_CABLE
- C27 pad 2: /PCB_Control/Amp_Control_Module_12/SPK_R_N -> +3.3V
- C270 pad 1: Net-(C270-Pad1) -> /Breakout_1/GND_LOCAL
- C270 pad 2: GND -> /Breakout_1/+5V_CABLE
- C271 pad 1: Net-(C271-Pad1) -> /Breakout_2/+1V8_LOCAL
- C271 pad 2: GND -> /Breakout_2/GND_LOCAL
- C272 pad 1: /PCB_Control/Amp_Control_Module_12/SPK_R_P -> /Breakout_2/GND_LOCAL
- C272 pad 2: GND -> /Breakout_2/+1V8_LOCAL
- C273 pad 1: GND -> /Breakout_2/+3.3V_LOCAL
- C273 pad 2: /PCB_Control/Amp_Control_Module_12/SPK_R_N -> /Breakout_2/GND_LOCAL
- C274 pad 1: Net-(C274-Pad1) -> /Breakout_2/+5V_CABLE
- C274 pad 2: GND -> /Breakout_2/GND_LOCAL
- C275 pad 1: Net-(C275-Pad1) -> /Breakout_2/GND_LOCAL
- C275 pad 2: GND -> /Breakout_2/+3.3V_LOCAL
- C276 pad 1: /PCB_Control/Amp_Control_Module_34/SPK_R_P -> /Breakout_2/+5V_CABLE
- C276 pad 2: GND -> /Breakout_2/GND_LOCAL
- C277 pad 1: GND -> /Breakout_2/GND_LOCAL
- C277 pad 2: /PCB_Control/Amp_Control_Module_34/SPK_R_N -> /Breakout_2/+1V8_LOCAL
- C278 pad 1: Net-(C278-Pad1) -> /Breakout_2/GND_LOCAL
- C278 pad 2: GND -> /Breakout_2/+5V_CABLE
- C279 pad 1: Net-(C279-Pad1) -> /Breakout_5/+1V8_LOCAL
- C279 pad 2: GND -> /Breakout_5/GND_LOCAL
- C28 pad 1: GND -> Net-(U14-CAPP)
- C28 pad 2: /PCB_Control/Amp_Control_Module_12/SPK_L_N -> Net-(U14-CAPM)
- C280 pad 1: /PCB_Control/Amp_Control_Module_56/SPK_R_P -> /Breakout_5/GND_LOCAL
- C280 pad 2: GND -> /Breakout_5/+1V8_LOCAL
- C281 pad 1: GND -> /Breakout_5/+3.3V_LOCAL
- C281 pad 2: /PCB_Control/Amp_Control_Module_56/SPK_R_N -> /Breakout_5/GND_LOCAL
- C282 pad 1: Net-(C282-Pad1) -> /Breakout_5/+5V_CABLE
- C282 pad 2: GND -> /Breakout_5/GND_LOCAL
- C283 pad 1: Net-(C283-Pad1) -> /Breakout_5/GND_LOCAL
- C283 pad 2: GND -> /Breakout_5/+3.3V_LOCAL
- C284 pad 1: /PCB_Control/Amp_Control_Module_78/SPK_R_P -> /Breakout_5/+5V_CABLE
- C284 pad 2: GND -> /Breakout_5/GND_LOCAL
- C285 pad 1: GND -> /Breakout_5/GND_LOCAL
- C285 pad 2: /PCB_Control/Amp_Control_Module_78/SPK_R_N -> /Breakout_5/+1V8_LOCAL
- C286 pad 1: Net-(C286-Pad1) -> /Breakout_5/GND_LOCAL
- C286 pad 2: GND -> /Breakout_5/+5V_CABLE
- C287 pad 1: Net-(C287-Pad1) -> /Breakout_1/+1V8_LOCAL
- C287 pad 2: GND -> /Breakout_1/GND_LOCAL
- C288 pad 1: +3.3V -> /Breakout_3/+1V8_LOCAL
- C288 pad 2: GND -> /Breakout_3/GND_LOCAL
- C29 pad 1: Net-(C29-Pad1) -> GND
- C29 pad 2: GND -> +3.3V
- C30 pad 1: Net-(C29-Pad1) -> GND
- C30 pad 2: /PCB_Control/Amp_Control_Module_12/LEFT_INPUT -> Net-(U14-LDOO)
- C31 pad 1: Net-(C31-Pad1) -> GND
- C31 pad 2: /PCB_Control/Amp_Control_Module_12/RIGHT_INPUT -> Net-(U14-VNEG)
- C32 pad 1: Net-(C31-Pad1) -> Net-(C32-Pad1)
- C33 pad 1: GND -> Net-(C32-Pad1)
- C33 pad 2: Net-(U11-LINN) -> /PCB_Control/Amp_Control_Module_12/LEFT_INPUT
- C34 pad 1: GND -> Net-(C34-Pad1)
- C34 pad 2: Net-(U55-LINN) -> /PCB_Control/Amp_Control_Module_12/RIGHT_INPUT
- C35 pad 1: /PCB_Control/Amp_Control_Module_12/VD_PLIMIT_R -> Net-(C34-Pad1)
- C36 pad 1: GND -> Net-(U15-GVDD)
- C36 pad 2: +24V -> GND
- C4 pad 1: GND -> +24V
- C4 pad 2: +24V -> GND
- C41 pad 1: GND -> /PCB_Control/Amp_Control_Module_12/W_BSPR
- C41 pad 2: +24V -> /PCB_Control/Amp_Control_Module_12/W_OUTPR
- C42 pad 1: /PCB_Control/Amp_Control_Module_34/W_BSPR -> /PCB_Control/Amp_Control_Module_12/W_BSNR
- C42 pad 2: /PCB_Control/Amp_Control_Module_34/W_OUTPR -> /PCB_Control/Amp_Control_Module_12/W_OUTNR
- C43 pad 1: /PCB_Control/Amp_Control_Module_34/W_BSNR -> /PCB_Control/Amp_Control_Module_12/W_BSPL
- C43 pad 2: /PCB_Control/Amp_Control_Module_34/W_OUTNR -> /PCB_Control/Amp_Control_Module_12/W_OUTPL
- C44 pad 1: /PCB_Control/Amp_Control_Module_34/W_BSPL -> /PCB_Control/Amp_Control_Module_12/W_BSNL
- C44 pad 2: /PCB_Control/Amp_Control_Module_34/W_OUTPL -> /PCB_Control/Amp_Control_Module_12/W_OUTNL
- C45 pad 1: /PCB_Control/Amp_Control_Module_34/W_BSNL -> GND
- C45 pad 2: /PCB_Control/Amp_Control_Module_34/W_OUTNL -> +24V
- C46 pad 1: Net-(U12-CAPP) -> GND
- C46 pad 2: Net-(U12-CAPM) -> +24V
- C47 pad 1: /PCB_Control/Amp_Control_Module_34/SPK_R_P -> GND
- C47 pad 2: /PCB_Control/Amp_Control_Module_34/SPK_R_N -> +24V
- C48 pad 1: /PCB_Control/Amp_Control_Module_34/SPK_L_P -> GND
- C48 pad 2: /PCB_Control/Amp_Control_Module_34/SPK_L_N -> +24V
- C49 pad 2: Net-(U12-LDOO) -> +24V
- C5 pad 2: Net-(U2-SS) -> +24V
- C50 pad 2: Net-(U12-VNEG) -> +24V
- C51 pad 1: GND -> /PCB_Control/Amp_Control_Module_12/SPK_R_P
- C51 pad 2: /PCB_Control/Amp_Control_Module_34/SPK_R_P -> /PCB_Control/Amp_Control_Module_12/SPK_R_N
- C52 pad 1: GND -> /PCB_Control/Amp_Control_Module_12/SPK_L_P
- C52 pad 2: /PCB_Control/Amp_Control_Module_34/SPK_L_P -> /PCB_Control/Amp_Control_Module_12/SPK_L_N
- C53 pad 2: /PCB_Control/Amp_Control_Module_34/SPK_R_N -> /PCB_Control/Amp_Control_Module_12/SPK_R_P
- C54 pad 2: /PCB_Control/Amp_Control_Module_34/SPK_L_N -> /PCB_Control/Amp_Control_Module_12/SPK_L_P
- C55 pad 1: Net-(C55-Pad1) -> GND
- C55 pad 2: GND -> /PCB_Control/Amp_Control_Module_12/SPK_R_N
- C56 pad 1: Net-(C55-Pad1) -> GND
- C56 pad 2: /PCB_Control/Amp_Control_Module_34/LEFT_INPUT -> /PCB_Control/Amp_Control_Module_12/SPK_L_N
- C57 pad 1: Net-(C57-Pad1) -> /PCB_Control/Amp_Control_Module_12/SPK_R_P
- C57 pad 2: /PCB_Control/Amp_Control_Module_34/RIGHT_INPUT -> GND
- C58 pad 1: Net-(C57-Pad1) -> GND
- C58 pad 2: GND -> /PCB_Control/Amp_Control_Module_12/SPK_R_N
- C59 pad 1: GND -> /PCB_Control/Amp_Control_Module_12/SPK_L_P
- C59 pad 2: Net-(U13-LINN) -> GND
- C6 pad 1: GND -> +24V
- C6 pad 2: Net-(U2-SW) -> GND
- C60 pad 2: Net-(U56-LINN) -> /PCB_Control/Amp_Control_Module_12/SPK_L_N
- C61 pad 1: Net-(U55-GVDD) -> /PCB_Control/Amp_Control_Module_12/VD_PLIMIT_R
- C62 pad 2: +24V -> Net-(U16-LINN)
- C63 pad 1: GND -> Net-(C63-Pad1)
- C63 pad 2: +24V -> GND
- C64 pad 1: GND -> Net-(C64-Pad1)
- C64 pad 2: +24V -> GND
- C65 pad 1: GND -> Net-(C65-Pad1)
- C65 pad 2: +24V -> GND
- C66 pad 1: GND -> Net-(C66-Pad1)
- C66 pad 2: +24V -> GND
- C67 pad 1: GND -> Net-(U16-GVDD)
- C67 pad 2: +24V -> GND
- C68 pad 1: /PCB_Control/Amp_Control_Module_56/W_BSPR -> GND
- C68 pad 2: /PCB_Control/Amp_Control_Module_56/W_OUTPR -> +24V
- C69 pad 1: /PCB_Control/Amp_Control_Module_56/W_BSNR -> GND
- C69 pad 2: /PCB_Control/Amp_Control_Module_56/W_OUTNR -> +24V
- C7 pad 1: +5V -> GND
- C7 pad 2: GND -> Net-(U2-SS)
- C70 pad 1: /PCB_Control/Amp_Control_Module_56/W_BSPL -> GND
- C70 pad 2: /PCB_Control/Amp_Control_Module_56/W_OUTPL -> +24V
- C71 pad 1: /PCB_Control/Amp_Control_Module_56/W_BSNL -> GND
- C71 pad 2: /PCB_Control/Amp_Control_Module_56/W_OUTNL -> +24V
- C72 pad 1: Net-(U14-CAPP) -> GND
- C72 pad 2: Net-(U14-CAPM) -> +24V
- C73 pad 1: /PCB_Control/Amp_Control_Module_56/SPK_R_P -> GND
- C73 pad 2: /PCB_Control/Amp_Control_Module_56/SPK_R_N -> +24V
- C74 pad 1: /PCB_Control/Amp_Control_Module_56/SPK_L_P -> GND
- C74 pad 2: /PCB_Control/Amp_Control_Module_56/SPK_L_N -> +24V
- C75 pad 2: Net-(U14-LDOO) -> +24V
- C76 pad 2: Net-(U14-VNEG) -> +24V
- C77 pad 2: /PCB_Control/Amp_Control_Module_56/SPK_R_P -> +24V
- C78 pad 2: /PCB_Control/Amp_Control_Module_56/SPK_L_P -> +3.3V
- C79 pad 2: /PCB_Control/Amp_Control_Module_56/SPK_R_N -> +3.3V
- C8 pad 1: +5V -> GND
- C8 pad 2: GND -> Net-(U2-SW)
- C80 pad 2: /PCB_Control/Amp_Control_Module_56/SPK_L_N -> +3.3V
- C81 pad 1: Net-(C81-Pad1) -> GND
- C82 pad 1: Net-(C81-Pad1) -> GND
- C82 pad 2: /PCB_Control/Amp_Control_Module_56/LEFT_INPUT -> +3.3V
- C83 pad 1: Net-(C83-Pad1) -> GND
- C83 pad 2: /PCB_Control/Amp_Control_Module_56/RIGHT_INPUT -> GND
- C84 pad 1: Net-(C83-Pad1) -> /PCB_Control/Amp_Control_Module_34/VD_PLIMIT_L
- C85 pad 2: Net-(U15-LINN) -> Net-(U18-LINN)
- C86 pad 2: Net-(U57-LINN) -> GND
- C87 pad 2: Net-(U58-LINN) -> +3.3V
- C88 pad 1: GND -> Net-(U17-CAPP)
- C88 pad 2: +24V -> Net-(U17-CAPM)
- C89 pad 2: +24V -> +3.3V
- C9 pad 1: GND -> +5V
- C9 pad 2: Net-(U3-EN) -> GND
- C90 pad 2: +24V -> Net-(U17-LDOO)
- C91 pad 2: +24V -> Net-(U17-VNEG)
- C92 pad 1: GND -> Net-(C92-Pad1)
- C92 pad 2: +24V -> GND
- C93 pad 1: GND -> Net-(C92-Pad1)
- C93 pad 2: +24V -> /PCB_Control/Amp_Control_Module_34/LEFT_INPUT
- C94 pad 1: /PCB_Control/Amp_Control_Module_78/W_BSPR -> Net-(C94-Pad1)
- C94 pad 2: /PCB_Control/Amp_Control_Module_78/W_OUTPR -> /PCB_Control/Amp_Control_Module_34/RIGHT_INPUT
- C95 pad 1: /PCB_Control/Amp_Control_Module_78/W_BSNR -> Net-(C94-Pad1)
- C95 pad 2: /PCB_Control/Amp_Control_Module_78/W_OUTNR -> GND
- C96 pad 1: /PCB_Control/Amp_Control_Module_78/W_BSPL -> Net-(U18-GVDD)
- C96 pad 2: /PCB_Control/Amp_Control_Module_78/W_OUTPL -> GND
- C97 pad 1: /PCB_Control/Amp_Control_Module_78/W_BSNL -> GND
- C97 pad 2: /PCB_Control/Amp_Control_Module_78/W_OUTNL -> +24V
- C98 pad 1: Net-(U16-CAPP) -> GND
- C98 pad 2: Net-(U16-CAPM) -> +24V
- C99 pad 1: /PCB_Control/Amp_Control_Module_78/SPK_R_P -> GND
- C99 pad 2: /PCB_Control/Amp_Control_Module_78/SPK_R_N -> +24V
- CN1 pad 3: GND -> unconnected-(CN1-Pad3)
- CN1 pad 4: GND -> unconnected-(CN1-Pad4)
- D4 pad 1: GND -> Net-(D4-K)
- D4 pad 2: +24V -> Net-(D4-A)
- D5 pad 1: +24V -> Net-(D4-K)
- D5 pad 2: Net-(D5-A) -> /PCB_Control/TEMP_OVERRIDE
- J10 pad 1: /PCB_Control/Amp_Control_Module_34/SPK_R_P -> /PCB_Control/Amp_Control_Module_78/SPK_L_P
- J10 pad 2: /PCB_Control/Amp_Control_Module_34/SPK_R_N -> /PCB_Control/Amp_Control_Module_78/SPK_L_N
- J11 pad 1: /PCB_Control/Amp_Control_Module_34/SPK_L_P -> /Breakout_4/+1V8_LOCAL
- J11 pad 2: /PCB_Control/Amp_Control_Module_34/SPK_L_N -> /Breakout_4/Breakout_Control/JUMPER
- J12 pad 1: /PCB_Control/Amp_Control_Module_56/SPK_R_P -> /Breakout_2/+1V8_LOCAL
- J12 pad 2: /PCB_Control/Amp_Control_Module_56/SPK_R_N -> /Breakout_2/Breakout_Control/JUMPER
- J13 pad 1: /PCB_Control/Amp_Control_Module_56/SPK_L_P -> /Breakout_5/+1V8_LOCAL
- J13 pad 2: /PCB_Control/Amp_Control_Module_56/SPK_L_N -> /Breakout_5/Breakout_Control/JUMPER
- J14 pad 1: /PCB_Control/Amp_Control_Module_78/SPK_R_P -> /Breakout_3/+1V8_LOCAL
- J14 pad 2: /PCB_Control/Amp_Control_Module_78/SPK_R_N -> /Breakout_3/Breakout_Control/JUMPER
- J15 pad 1: /PCB_Control/Amp_Control_Module_78/SPK_L_P -> /Breakout_1/+1V8_LOCAL
- J15 pad 2: /PCB_Control/Amp_Control_Module_78/SPK_L_N -> /Breakout_1/Breakout_Control/JUMPER
- J16 pad 1: /Breakout_4/+1V8_LOCAL -> /Breakout_6/+1V8_LOCAL
- J16 pad 2: /Breakout_4/Breakout_Control/JUMPER -> /Breakout_6/Breakout_Control/JUMPER
- J16 pad 3: /Breakout_4/GND_LOCAL -> /Breakout_6/GND_LOCAL
- J3 pad 1: I2S_BCLK -> /PCB_Control/Amp_Control_Module_12/SPK_R_P
- J3 pad 2: I2S_LRCK -> /PCB_Control/Amp_Control_Module_12/SPK_R_N
- J8 pad 1: /PCB_Control/Amp_Control_Module_12/SPK_R_P -> /PCB_Control/Amp_Control_Module_56/SPK_L_P
- J8 pad 2: /PCB_Control/Amp_Control_Module_12/SPK_R_N -> /PCB_Control/Amp_Control_Module_56/SPK_L_N
- J9 pad 1: /PCB_Control/Amp_Control_Module_12/SPK_L_P -> /PCB_Control/Amp_Control_Module_78/SPK_R_P
- J9 pad 2: /PCB_Control/Amp_Control_Module_12/SPK_L_N -> /PCB_Control/Amp_Control_Module_78/SPK_R_N
- Q1 pad 1: Net-(D6-K) -> Net-(D4-K)
- Q1 pad 3: Net-(D5-A) -> Net-(D2-A)
- R10 pad 1: /Hub_Main/Hub_Mic_Module_4/DATA_N -> Net-(U15-AVCC)
- R10 pad 2: /Hub_Main/Hub_Mic_Module_4/DATA_P -> +24V
- R11 pad 1: Net-(C264-Pad1) -> GND
- R11 pad 2: /PCB_Control/Amp_Control_Module_12/SPK_L_N -> /PCB_Control/Amp_Control_Module_12/VD_PLIMIT_L
- R12 pad 1: Net-(C265-Pad1) -> Net-(U15-GVDD)
- R12 pad 2: /PCB_Control/Amp_Control_Module_34/SPK_L_N -> /PCB_Control/Amp_Control_Module_12/GAIN_SET_L
- R13 pad 1: Net-(C266-Pad1) -> GND
- R13 pad 2: /PCB_Control/Amp_Control_Module_56/SPK_L_N -> /PCB_Control/Amp_Control_Module_12/GAIN_SET_L
- R14 pad 1: Net-(U10-OUTL) -> /PCB_Control/AMP_FAULT_1
- R14 pad 2: Net-(C29-Pad1) -> +3.3V
- R15 pad 1: Net-(U10-OUTR) -> /PCB_Control/Amp_Control_Module_12/SPK_R_P
- R15 pad 2: Net-(C31-Pad1) -> Net-(C63-Pad1)
- R16 pad 1: Net-(U11-AVCC) -> Net-(C64-Pad1)
- R16 pad 2: +24V -> /PCB_Control/Amp_Control_Module_12/SPK_R_N
- R17 pad 1: /PCB_Control/AMP_FAULT_1 -> /PCB_Control/Amp_Control_Module_12/SPK_L_P
- R17 pad 2: +3.3V -> Net-(C65-Pad1)
- R18 pad 1: Net-(C267-Pad1) -> Net-(C66-Pad1)
- R18 pad 2: /PCB_Control/Amp_Control_Module_78/SPK_L_N -> /PCB_Control/Amp_Control_Module_12/SPK_L_N
- R19 pad 1: /PCB_Control/Amp_Control_Module_12/SPK_L_P -> /PCB_Control/Amp_Control_Module_12/VD_PLIMIT_R
- R19 pad 2: Net-(C268-Pad1) -> Net-(U16-GVDD)
- R20 pad 1: /PCB_Control/Amp_Control_Module_34/SPK_L_P -> Net-(U16-AVCC)
- R20 pad 2: Net-(C269-Pad1) -> +24V
- R21 pad 1: Net-(U12-OUTL) -> GND
- R21 pad 2: Net-(C55-Pad1) -> /PCB_Control/Amp_Control_Module_12/VD_PLIMIT_R
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