File: diff_hub.kicad_sch (KiCad schematic)
At the start: 4 parts, among them U5 MAX3485_SC, U6 MAX3485_WS

Commit message: Fixed most ERC checks
Parts:
- renumbered C8 to C10, C9 to C11, U5 to U4, U6 to U5
Connections:
- no-connect marks 0 -> 2
Changed lines of the file:
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@@
 		(color 0 0 0 0)
+	)
+	(no_connect
+		(at 87.63 40.64)
+	)
+	(no_connect
+		(at 36.83 40.64)
 	)
 	(wire
@@
 		(dnp no)
 		(fields_autoplaced yes)
-		(property "Reference" "U6"
+		(property "Reference" "U5"
 			(at 99.9333 27.94 0)
 			(effects
@@
 			(project "AEC_Speaker_Mic_System"
 				(path "/b4ee80b5-9d9a-4551-9b0c-6a8cb8d78ca3/ff66f788-06df-4fa5-89ad-7a9539b69b02"
-					(reference "U6")
+					(reference "U5")
 					(unit 1)
 				)
@@
 		(dnp no)
 		(fields_autoplaced yes)
-		(property "Reference" "#PWR023"
+		(property "Reference" "#PWR030"
 			(at 40.64 43.18 0)
 			(effects
@@
 			(project "AEC_Speaker_Mic_System"
 				(path "/b4ee80b5-9d9a-4551-9b0c-6a8cb8d78ca3/ff66f788-06df-4fa5-89ad-7a9539b69b02"
-					(reference "#PWR023")
+					(reference "#PWR030")
 					(unit 1)
 				)
@@
 		(dnp no)
 		(fields_autoplaced yes)
-		(property "Reference" "#PWR024"
+		(property "Reference" "#PWR031"
 			(at 40.64 45.72 0)
 			(effects
@@
 			(project "AEC_Speaker_Mic_System"
 				(path "/b4ee80b5-9d9a-4551-9b0c-6a8cb8d78ca3/ff66f788-06df-4fa5-89ad-7a9539b69b02"
-					(reference "#PWR024")
+					(reference "#PWR031")
 					(unit 1)
 				)
@@
 		(dnp no)
 		(fields_autoplaced yes)
-		(property "Reference" "#PWR026"
+		(property "Reference" "#PWR036"
 			(at 91.44 45.72 0)
 			(effects
@@
 			(project "AEC_Speaker_Mic_System"
 				(path "/b4ee80b5-9d9a-4551-9b0c-6a8cb8d78ca3/ff66f788-06df-4fa5-89ad-7a9539b69b02"
-					(reference "#PWR026")
+					(reference "#PWR036")
 					(unit 1)
 				)
@@
 		(dnp no)
 		(fields_autoplaced yes)
-		(property "Reference" "#PWR027"
+		(property "Reference" "#PWR033"
 			(at 46.99 67.31 0)
 			(effects
@@
 			(project "AEC_Speaker_Mic_System"
 				(path "/b4ee80b5-9d9a-4551-9b0c-6a8cb8d78ca3/ff66f788-06df-4fa5-89ad-7a9539b69b02"
-					(reference "#PWR027")
+					(reference "#PWR033")
 					(unit 1)
 				)
@@
 		(dnp no)
 		(fields_autoplaced yes)
-		(property "Reference" "C8"
+		(property "Reference" "C10"
 			(at 44.45 25.3999 0)
 			(effects
@@
 			(project "AEC_Speaker_Mic_System"
 				(path "/b4ee80b5-9d9a-4551-9b0c-6a8cb8d78ca3/ff66f788-06df-4fa5-89ad-7a9539b69b02"
-					(reference "C8")
+					(reference "C10")
 					(unit 1)
 				)
@@
 		(dnp no)
 		(fields_autoplaced yes)
-		(property "Reference" "#PWR028"
+		(property "Reference" "#PWR038"
 			(at 97.79 67.31 0)
 			(effects
@@
 			(project "AEC_Speaker_Mic_System"
 				(path "/b4ee80b5-9d9a-4551-9b0c-6a8cb8d78ca3/ff66f788-06df-4fa5-89ad-7a9539b69b02"
-					(reference "#PWR028")
+					(reference "#PWR038")
 					(unit 1)
 				)
@@
 		(dnp no)
 		(fields_autoplaced yes)
-		(property "Reference" "#PWR032"
+		(property "Reference" "#PWR037"
 			(at 97.79 22.86 0)
 			(effects
@@
 			(project "AEC_Speaker_Mic_System"
 				(path "/b4ee80b5-9d9a-4551-9b0c-6a8cb8d78ca3/ff66f788-06df-4fa5-89ad-7a9539b69b02"
-					(reference "#PWR032")
+					(reference "#PWR037")
 					(unit 1)
 				)
@@
 		(dnp no)
 		(fields_autoplaced yes)
-		(property "Reference" "#PWR030"
+		(property "Reference" "#PWR034"
 			(at 85.09 34.29 0)
 			(effects
@@
 			(project "AEC_Speaker_Mic_System"
 				(path "/b4ee80b5-9d9a-4551-9b0c-6a8cb8d78ca3/ff66f788-06df-4fa5-89ad-7a9539b69b02"
-					(reference "#PWR030")
+					(reference "#PWR034")
 					(unit 1)
 				)
@@
 		(dnp no)
 		(fields_autoplaced yes)
-		(property "Reference" "U5"
+		(property "Reference" "U4"
 			(at 49.1333 27.94 0)
 			(effects
@@
 			(project "AEC_Speaker_Mic_System"
 				(path "/b4ee80b5-9d9a-4551-9b0c-6a8cb8d78ca3/ff66f788-06df-4fa5-89ad-7a9539b69b02"
-					(reference "U5")
+					(reference "U4")
 					(unit 1)
 				)
@@
 		(dnp no)
 		(fields_autoplaced yes)
-		(property "Reference" "#PWR025"
+		(property "Reference" "#PWR035"
 			(at 91.44 43.18 0)
 			(effects
@@
 			(project "AEC_Speaker_Mic_System"
 				(path "/b4ee80b5-9d9a-4551-9b0c-6a8cb8d78ca3/ff66f788-06df-4fa5-89ad-7a9539b69b02"
-					(reference "#PWR025")
+					(reference "#PWR035")
 					(unit 1)
 				)
@@
 		(dnp no)
 		(fields_autoplaced yes)
-		(property "Reference" "#PWR031"
+		(property "Reference" "#PWR032"
 			(at 46.99 22.86 0)
 			(effects
@@
 			(project "AEC_Speaker_Mic_System"
 				(path "/b4ee80b5-9d9a-4551-9b0c-6a8cb8d78ca3/ff66f788-06df-4fa5-89ad-7a9539b69b02"
-					(reference "#PWR031")
+					(reference "#PWR032")
 					(unit 1)
 				)
@@
 		(dnp no)
 		(fields_autoplaced yes)
-		(property "Reference" "C9"
+		(property "Reference" "C11"
 			(at 95.25 25.3999 0)
 			(effects
@@
 			(project "AEC_Speaker_Mic_System"
 				(path "/b4ee80b5-9d9a-4551-9b0c-6a8cb8d78ca3/ff66f788-06df-4fa5-89ad-7a9539b69b02"
-					(reference "C9")
+					(reference "C11")
 					(unit 1)
 				)

Commit message: Footprinting done (warnings on schematic side but pcb import works fine)
Parts:
- C10, C11: footprint (none) -> Capacitor_SMD:C_0603_1608Metric
Changed lines of the file:
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@@
 			)
 		)
-		(property "Footprint" ""
+		(property "Footprint" "Capacitor_SMD:C_0603_1608Metric"
 			(at 41.6052 30.48 0)
 			(effects
@@
 			)
 		)
-		(property "Footprint" ""
+		(property "Footprint" "Capacitor_SMD:C_0603_1608Metric"
 			(at 92.4052 30.48 0)
 			(effects

Commit message: Minor schematic changes
Parts:
- renumbered C10 to C12, C11 to C13
Changed lines of the file:
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@@
 		(dnp no)
 		(fields_autoplaced yes)
-		(property "Reference" "#PWR030"
+		(property "Reference" "#PWR034"
 			(at 40.64 43.18 0)
 			(effects
@@
 			(project "AEC_Speaker_Mic_System"
 				(path "/b4ee80b5-9d9a-4551-9b0c-6a8cb8d78ca3/ff66f788-06df-4fa5-89ad-7a9539b69b02"
-					(reference "#PWR030")
+					(reference "#PWR034")
 					(unit 1)
 				)
@@
 		(dnp no)
 		(fields_autoplaced yes)
-		(property "Reference" "#PWR031"
+		(property "Reference" "#PWR035"
 			(at 40.64 45.72 0)
 			(effects
@@
 			(project "AEC_Speaker_Mic_System"
 				(path "/b4ee80b5-9d9a-4551-9b0c-6a8cb8d78ca3/ff66f788-06df-4fa5-89ad-7a9539b69b02"
-					(reference "#PWR031")
+					(reference "#PWR035")
 					(unit 1)
 				)
@@
 		(dnp no)
 		(fields_autoplaced yes)
-		(property "Reference" "#PWR036"
+		(property "Reference" "#PWR040"
 			(at 91.44 45.72 0)
 			(effects
@@
 			(project "AEC_Speaker_Mic_System"
 				(path "/b4ee80b5-9d9a-4551-9b0c-6a8cb8d78ca3/ff66f788-06df-4fa5-89ad-7a9539b69b02"
-					(reference "#PWR036")
+					(reference "#PWR040")
 					(unit 1)
 				)
@@
 		(dnp no)
 		(fields_autoplaced yes)
-		(property "Reference" "#PWR033"
+		(property "Reference" "#PWR037"
 			(at 46.99 67.31 0)
 			(effects
@@
 			(project "AEC_Speaker_Mic_System"
 				(path "/b4ee80b5-9d9a-4551-9b0c-6a8cb8d78ca3/ff66f788-06df-4fa5-89ad-7a9539b69b02"
-					(reference "#PWR033")
+					(reference "#PWR037")
 					(unit 1)
 				)
@@
 		(dnp no)
 		(fields_autoplaced yes)
-		(property "Reference" "C10"
+		(property "Reference" "C12"
 			(at 44.45 25.3999 0)
 			(effects
@@
 			(project "AEC_Speaker_Mic_System"
 				(path "/b4ee80b5-9d9a-4551-9b0c-6a8cb8d78ca3/ff66f788-06df-4fa5-89ad-7a9539b69b02"
-					(reference "C10")
+					(reference "C12")
 					(unit 1)
 				)
@@
 		(dnp no)
 		(fields_autoplaced yes)
-		(property "Reference" "#PWR038"
+		(property "Reference" "#PWR042"
 			(at 97.79 67.31 0)
 			(effects
@@
 			(project "AEC_Speaker_Mic_System"
 				(path "/b4ee80b5-9d9a-4551-9b0c-6a8cb8d78ca3/ff66f788-06df-4fa5-89ad-7a9539b69b02"
-					(reference "#PWR038")
+					(reference "#PWR042")
 					(unit 1)
 				)
@@
 		(dnp no)
 		(fields_autoplaced yes)
-		(property "Reference" "#PWR037"
+		(property "Reference" "#PWR041"
 			(at 97.79 22.86 0)
 			(effects
@@
 			(project "AEC_Speaker_Mic_System"
 				(path "/b4ee80b5-9d9a-4551-9b0c-6a8cb8d78ca3/ff66f788-06df-4fa5-89ad-7a9539b69b02"
-					(reference "#PWR037")
+					(reference "#PWR041")
 					(unit 1)
 				)
@@
 		(dnp no)
 		(fields_autoplaced yes)
-		(property "Reference" "#PWR034"
+		(property "Reference" "#PWR038"
 			(at 85.09 34.29 0)
 			(effects
@@
 			(project "AEC_Speaker_Mic_System"
 				(path "/b4ee80b5-9d9a-4551-9b0c-6a8cb8d78ca3/ff66f788-06df-4fa5-89ad-7a9539b69b02"
-					(reference "#PWR034")
+					(reference "#PWR038")
 					(unit 1)
 				)
@@
 		(dnp no)
 		(fields_autoplaced yes)
-		(property "Reference" "#PWR029"
+		(property "Reference" "#PWR033"
 			(at 34.29 34.29 0)
 			(effects
@@
 			(project "AEC_Speaker_Mic_System"
 				(path "/b4ee80b5-9d9a-4551-9b0c-6a8cb8d78ca3/ff66f788-06df-4fa5-89ad-7a9539b69b02"
-					(reference "#PWR029")
+					(reference "#PWR033")
 					(unit 1)
 				)
@@
 		(dnp no)
 		(fields_autoplaced yes)
-		(property "Reference" "#PWR035"
+		(property "Reference" "#PWR039"
 			(at 91.44 43.18 0)
 			(effects
@@
 			(project "AEC_Speaker_Mic_System"
 				(path "/b4ee80b5-9d9a-4551-9b0c-6a8cb8d78ca3/ff66f788-06df-4fa5-89ad-7a9539b69b02"
-					(reference "#PWR035")
+					(reference "#PWR039")
 					(unit 1)
 				)
@@
 		(dnp no)
 		(fields_autoplaced yes)
-		(property "Reference" "#PWR032"
+		(property "Reference" "#PWR036"
 			(at 46.99 22.86 0)
 			(effects
@@
 			(project "AEC_Speaker_Mic_System"
 				(path "/b4ee80b5-9d9a-4551-9b0c-6a8cb8d78ca3/ff66f788-06df-4fa5-89ad-7a9539b69b02"
-					(reference "#PWR032")
+					(reference "#PWR036")
 					(unit 1)
 				)
@@
 		(dnp no)
 		(fields_autoplaced yes)
-		(property "Reference" "C11"
+		(property "Reference" "C13"
 			(at 95.25 25.3999 0)
 			(effects
@@
 			(project "AEC_Speaker_Mic_System"
 				(path "/b4ee80b5-9d9a-4551-9b0c-6a8cb8d78ca3/ff66f788-06df-4fa5-89ad-7a9539b69b02"
-					(reference "C11")
-					(unit 1)
-				)
+					(reference "C13")
+					(unit 1)
+				)
